Commit message: Merged

File: robo_spawn/urdf/turtlebot3_waffle_pi.urdf.xacro (robot description, xacro)
@@ -161,5 +161,5 @@
   </link>
   <joint name="camera_joint" type="fixed">
-    <origin xyz="0.073 -0.011 0.300" rpy="0 0 0"/>
+    <origin xyz="0.073 -0.011 0.350" rpy="0 0 0"/>
     <parent link="base_link"/>
     <child link="camera_link"/>
